Commit message: Result improve commit

File: catkin_ws/src/turtlebot3/turtlebot3_description/urdf/turtlebot3_waffle.urdf.xacro (robot description, xacro)
@@ -137,5 +137,5 @@
   </joint>
   <link name="imu_link"/>
-<!-- laser  -->
+<!-- laser
   <joint name="scan_joint" type="fixed">
     <parent link="base_link"/>
@@ -164,5 +164,5 @@
                izz="0.001" />
     </inertial>
-  </link>
+  </link>-->
   <joint name="camera_joint" type="fixed">
     <origin xyz="0.064 -0.065 0.094" rpy="0 0 0"/>
@@ -216,7 +216,7 @@
   </joint>
   <link name="camera_depth_optical_frame"/>
-  <!-- <xacro:include filename="$(find velodyne_description)/urdf/VLP-16.urdf.xacro"/>
+  <xacro:include filename="$(find velodyne_description)/urdf/VLP-16.urdf.xacro"/>
   <xacro:VLP-16 parent="base_link" name="velodyne" topic="/velodyne_points" hz="10" samples="360" gpu="false" min_angle="-1.57" max_angle="1.57" min_range="0.1">
     <origin xyz="-0.064 0 0.122" rpy="0 0 0" />
-  </xacro:VLP-16> -->
+  </xacro:VLP-16>
 </robot>

File: catkin_ws/src/turtlebot3/turtlebot3_description/urdf/turtlebot3_waffle_pi.gazebo.xacro (robot description, xacro)
@@ -113,13 +113,13 @@
         <scan>
           <horizontal>
-            <samples>360</samples>
+            <samples>120</samples>
             <resolution>1</resolution>
-            <min_angle>0.0</min_angle>
-            <max_angle>6.28319</max_angle>
+            <min_angle>0</min_angle>
+            <max_angle>6.283185</max_angle>
           </horizontal>
         </scan>
         <range>
-          <min>0.120</min>
-          <max>3.5</max>
+          <min>0.160</min>
+          <max>8</max>
           <resolution>0.015</resolution>
         </range>

File: catkin_ws/src/turtlebot3/turtlebot3_description/urdf/turtlebot3_waffle_pi.urdf.xacro (robot description, xacro)
@@ -133,5 +133,5 @@
   </joint>
   <link name="imu_link"/>
-  <!-- laser
+  <!-- laser  -->
   <joint name="scan_joint" type="fixed">
     <parent link="base_link"/>
@@ -160,5 +160,5 @@
                izz="0.001" />
     </inertial>
-  </link>-->
+  </link>
   <joint name="camera_joint" type="fixed">
     <origin xyz="0.073 -0.011 0.084" rpy="0 0 0"/>
@@ -186,7 +186,7 @@
   </joint>
   <link name="camera_rgb_optical_frame"/>
-  <xacro:include filename="$(find velodyne_description)/urdf/VLP-16.urdf.xacro"/>
+  <!-- <xacro:include filename="$(find velodyne_description)/urdf/VLP-16.urdf.xacro"/>
   <xacro:VLP-16 parent="base_link" name="velodyne" topic="/velodyne_points" hz="10" samples="360" gpu="false" min_angle="-1.57" max_angle="1.57" min_range="0.1">
     <origin xyz="-0.064 0 0.122" rpy="0 0 0" />
-  </xacro:VLP-16>
+  </xacro:VLP-16> -->
 </robot>
